File: hardware/power_output.kicad_sch (KiCad schematic)
At the start: 0 parts

Commit message: Need to revisit current limitation (use PWM), need to use charge pump for CCM of output drivers
Parts:
- added C48, C49: 390p, symbol Device:C
- added C50: C_Small, symbol Device:C_Small
- added C51: C, symbol Device:C
- added D3: SSB44, PCM_Diode_SMD_AKL:D_SMB, symbol PCM_Diode_Schottky_AKL:SSB44
- added D4: TPSMC20A, PCM_Diode_SMD_AKL:D_SMC, symbol PCM_Diode_TVS_AKL:TPSMC20A
- added Q1: IAUCN04S7N056D, openvcu:Infineon_PG-TDSON-8-61_ThermalVias, symbol Transistor_FET:Q_Dual_NMOS_S1G1S2G2D2D2D1D1
- added R10: 10m, symbol Device:R
- added R6, R8: 10, symbol Device:R
- added R9: 2R2, symbol Device:R
- added U15: UCC27735-Q1, Package_SO:SOIC-14_3.9x8.7mm_P1.27mm, symbol openvcu:UCC27735-Q1
Connections:
- new net: C48.1, R6.2, U15.1 (HI)
- new net: U15.10 (NC), U15.14 (NC), U15.8 (NC), U15.9 (NC)
- new net: C50.2, U15.11 (HS)
- new net: Q1.4 (G), U15.12 (HO)
- new net: C50.1, D3.1 (K), U15.13 (HB)
- new net: C49.1, R8.2, U15.2 (LI)
- new net: Q1.2 (G), U15.6 (LO)
- new net: C51.1, R9.1, U15.7 (VDD)
- new net: Q1.3 (S), Q1.7 (D), Q1.8 (D), R10.1
- new net: D3.2 (A), R9.2
- new net +12VBAT: Q1.5 (D), Q1.6 (D)
- new net EN: U15.4 (EN/NC)
- new net GND: C48.2, C49.2, C51.2, D4.2 (A), Q1.1 (S), U15.3 (VSS), U15.5 (COM)
- new net HI: R6.1
- new net LI: R8.1
- new net OUT: D4.1 (K), R10.2
